Commit message: change default setting of realsense& urdf_file

File: src/mybot_moveit_config/config/gazebo_myur5.urdf (robot description, URDF)
Before this commit: robot myur5, 49 links, 48 joints
Links:
- added link camera_accel_frame
- added link camera_accel_optical_frame
- added link camera_color_frame
- added link camera_color_optical_frame
- added link camera_depth_frame
- added link camera_depth_optical_frame
- added link camera_gyro_frame
- added link camera_gyro_optical_frame
- added link camera_infra1_frame
- added link camera_infra1_optical_frame
- added link camera_infra2_frame
- added link camera_infra2_optical_frame
Joints:
- added joint camera_accel_joint: type fixed, parent camera_link, child camera_accel_frame, origin xyz=-0.01174 -0.00552 0.0051 rpy=0 0 0
- added joint camera_accel_optical_joint: type fixed, parent camera_accel_frame, child camera_accel_optical_frame, origin xyz=0 0 0 rpy=-1.5707963267948966 0 -1.5707963267948966
- added joint camera_color_joint: type fixed, parent camera_link, child camera_color_frame, origin xyz=0 0.015 0 rpy=0 0 0
- added joint camera_color_optical_joint: type fixed, parent camera_color_frame, child camera_color_optical_frame, origin xyz=0 0 0 rpy=-1.5707963267948966 0 -1.5707963267948966
- added joint camera_depth_joint: type fixed, parent camera_link, child camera_depth_frame, origin xyz=0 0 0 rpy=0 0 0
- added joint camera_depth_optical_joint: type fixed, parent camera_depth_frame, child camera_depth_optical_frame, origin xyz=0 0 0 rpy=-1.5707963267948966 0 -1.5707963267948966
- added joint camera_gyro_joint: type fixed, parent camera_link, child camera_gyro_frame, origin xyz=-0.01174 -0.00552 0.0051 rpy=0 0 0
- added joint camera_gyro_optical_joint: type fixed, parent camera_gyro_frame, child camera_gyro_optical_frame, origin xyz=0 0 0 rpy=-1.5707963267948966 0 -1.5707963267948966
- added joint camera_infra1_joint: type fixed, parent camera_link, child camera_infra1_frame, origin xyz=0 0.0 0 rpy=0 0 0
- added joint camera_infra1_optical_joint: type fixed, parent camera_infra1_frame, child camera_infra1_optical_frame, origin xyz=0 0 0 rpy=-1.5707963267948966 0 -1.5707963267948966
- added joint camera_infra2_joint: type fixed, parent camera_link, child camera_infra2_frame, origin xyz=0 -0.05 0 rpy=0 0 0
- added joint camera_infra2_optical_joint: type fixed, parent camera_infra2_frame, child camera_infra2_optical_frame, origin xyz=0 0 0 rpy=-1.5707963267948966 0 -1.5707963267948966

File: src/realsense-ros/realsense2_description/urdf/_d435i.urdf.xacro (robot description, xacro)
@@ -9,5 +9,5 @@
   <xacro:include filename="$(find realsense2_description)/urdf/_d435.urdf.xacro"/>
   <xacro:include filename="$(find realsense2_description)/urdf/_d435i_imu_modules.urdf.xacro"/>
-  <xacro:macro name="sensor_d435i" params="parent *origin name:=camera use_nominal_extrinsics:=false add_plug:=false topics_ns:=camera publish_pointcloud:=false" >
+  <xacro:macro name="sensor_d435i" params="parent *origin name:=camera use_nominal_extrinsics:=true add_plug:=false topics_ns:=camera publish_pointcloud:=true" >
     <xacro:sensor_d435 parent="${parent}" name="${name}" use_nominal_extrinsics="${use_nominal_extrinsics}" add_plug="${add_plug}" topics_ns="${topics_ns}" publish_pointcloud="${publish_pointcloud}">
       <xacro:insert_block name="origin" />

File: src/realsense-ros/realsense2_description/urdf/test_d435i_camera.urdf.xacro (robot description, xacro)
@@ -3,5 +3,5 @@
   <xacro:arg name="name" default="camera" />
   <xacro:arg name="topics_ns" default="camera" />
-  <xacro:arg name="use_nominal_extrinsics" default="false" />
+  <xacro:arg name="use_nominal_extrinsics" default="true" />
   <xacro:arg name="publish_pointcloud" default="false" />
   <xacro:arg name="add_plug" default="false" />

Commit message: modify some interial parameters of the ur
description

File: src/mybot_moveit_config/config/gazebo_myur5.urdf (robot description, URDF)
Before this commit: robot myur5, 61 links, 60 joints
Links:
- link ft300_mounting_plate: mass 0.1 -> 0.072
- link ft300_sensor: mass 0.300 -> 0.00
Joints:
- joint shoulder_pan_joint: limit lower=-6.283185307179586 upper=6.283185307179586 effort=150.0 velocity=3.141592653589793 -> lower=-6.283185307179586 upper=6.283185307179586 effort=200.0 velocity=3.141592653589793
- joint wrist_1_joint: limit lower=-6.283185307179586 upper=6.283185307179586 effort=28.0 velocity=3.141592653589793 -> lower=-6.283185307179586 upper=6.283185307179586 effort=150.0 velocity=3.141592653589793
- joint wrist_2_joint: limit lower=-6.283185307179586 upper=6.283185307179586 effort=28.0 velocity=3.141592653589793 -> lower=-6.283185307179586 upper=6.283185307179586 effort=60.0 velocity=3.141592653589793
- joint wrist_3_joint: limit lower=-6.283185307179586 upper=6.283185307179586 effort=28.0 velocity=3.141592653589793 -> lower=-6.283185307179586 upper=6.283185307179586 effort=5000.0 velocity=3.141592653589793
