Commit message: Change the base mass of MiR250 for simulation
Change the base mass of MiR250 for simulation

File: src/mir_robot/mir_description/urdf/include/mir_v1.urdf.xacro (robot description, xacro)
@@ -27,5 +27,5 @@
   </xacro:if>
   <xacro:if value="${mir_type == 'mir_250'}">
-    <xacro:property name="mir_base_mass" value="97.0" />
+    <xacro:property name="mir_base_mass" value="1997.0" />
     <xacro:property name="mir_act_wheel_radius" value="0.100" />
     <xacro:property name="mir_act_wheel_width" value="0.038" />

Commit message: Add files via upload

File: src/mir_robot/mir_description/urdf/include/mir_v1.urdf.xacro (robot description, xacro)
@@ -27,5 +27,5 @@
   </xacro:if>
   <xacro:if value="${mir_type == 'mir_250'}">
-    <xacro:property name="mir_base_mass" value="1997.0" />
+    <xacro:property name="mir_base_mass" value="997.0" />
     <xacro:property name="mir_act_wheel_radius" value="0.100" />
     <xacro:property name="mir_act_wheel_width" value="0.038" />
@@ -59,5 +59,5 @@
     <xacro:property name="laser_dy" value="0.205" />
   </xacro:if>
-  <xacro:property name="laser_dz" value="0.1914" />
+  <xacro:property name="laser_dz" value="0.183" />
   <xacro:macro name="actuated_wheel" params="prefix locationprefix locationright">
     <joint name="${prefix}${locationprefix}_wheel_joint" type="continuous">
@@ -196,4 +196,12 @@
           <mesh filename="package://mir_description/meshes/collision/${mir_type}_base.stl" />
         </geometry>
+        <surface>
+          <friction>
+            <ode>
+              <mu>119.91</mu>
+              <mu2>119.91</mu2>
+            </ode>
+          </friction>
+        </surface>
       </collision>
     </link>
