Commit message: Add files via upload

File: src/myur_description/urdf/myur5.urdf.xacro (robot description, xacro)
@@ -32,5 +32,5 @@
         <parent link="world"/>
         <child link="table"/>
-        <origin xyz="0.0 0.0 0.0" rpy="0.0 0.0 0.0"/>
+        <origin xyz="0.0 0.0 0.1" rpy="0.0 0.0 0.0"/>
     </joint>
     <xacro:include filename="$(find ur_description)/urdf/inc/ur_common.xacro" />

Commit message: src
add the force&torque sensor

File: src/myur_description/urdf/myur5.urdf.xacro (robot description, xacro)
@@ -40,10 +40,14 @@
         <child link="base_link"/>
     </joint>
+    <xacro:include filename="$(find robotiq_ft_sensor)/urdf/robotiq_ft300.urdf.xacro" />
+    <xacro:robotiq_ft300 prefix="" parent="tool0">
+      <origin xyz="0 0 0" rpy="0 0 0"/>
+    </xacro:robotiq_ft300>
     <xacro:include filename="$(find robotiq_2f_140_gripper_visualization)/urdf/robotiq_arg2f_140_model.xacro" />
-    <joint name="end_effector_joint" type="fixed">
-        <origin xyz="0.0 0.0 0.0" rpy="0.0 0.0 0.0"/>
-        <parent link="wrist_3_link"/>
+    <joint name="ft_gripper_joint" type="fixed">
+        <parent link="robotiq_ft_frame_id"/>
         <child link="robotiq_arg2f_base_link"/>
-    </joint>
+        <origin xyz="0 0 0" rpy="0 0 0"/>
+      </joint>
 <!-- Gazebo plugin for ROS Control -->
   <gazebo>

Commit message: src
add camera holder& camera

File: src/myur_description/urdf/myur5.urdf.xacro (robot description, xacro)
@@ -37,6 +37,17 @@
       <origin xyz="0 0 0" rpy="0 0 0"/>
     </xacro:robotiq_ft300>
+    <xacro:include filename="$(find camera_holder)/urdf/camera_holder.urdf" />
+    <joint name="camera_holder_joint" type="fixed">
+        <parent link="wrist_3_link"/>
+        <child link="camera_holder_link"/>
+        <origin xyz="-0.0395 0 -0.03" rpy="1.5708 0 1.5708"/>
+      </joint>
+      <xacro:arg name="use_nominal_extrinsics" default="false" />
+      <xacro:include filename="$(find realsense2_description)/urdf/_d435i.urdf.xacro"/>
+      <xacro:sensor_d435i parent="camera_holder_link" use_nominal_extrinsics="$(arg use_nominal_extrinsics)">
+      <origin xyz="-0.11 0.026 0.04" rpy="-1.5708 0 1.5708"/>
+      </xacro:sensor_d435i>
     <xacro:include filename="$(find robotiq_2f_140_gripper_visualization)/urdf/robotiq_arg2f_140_model.xacro" />
-    <joint name="ft_gripper_joint" type="fixed">
+      <joint name="ft_gripper_joint" type="fixed">
         <parent link="robotiq_ft_frame_id"/>
         <child link="robotiq_arg2f_base_link"/>

Commit message: Update myur5.urdf.xacro

File: src/myur_description/urdf/myur5.urdf.xacro (robot description, xacro)
@@ -4,5 +4,5 @@
     <xacro:include filename="$(find booksink)/urdf/booksink.urdf"/>
     <joint name="mir_sink_joint" type="fixed">
-        <parent link="mir_base_link"/>
+        <parent link="mir/base_link"/>
         <child link="booksink_link"/>
         <origin xyz="-0.38478 0.285055 0.2964" rpy="0.0 0.0 0.0"/>
@@ -24,5 +24,5 @@
     <joint name="mass_joint" type="fixed">
         <origin xyz="0 0 0.1" rpy="0.0 0.0 0.0"/>
-        <parent link="mir_base_link"/>
+        <parent link="mir/base_link"/>
         <child link="mass_link"/>
     </joint>

Commit message: Add files via upload
updated myur configuration

File: src/myur_description/urdf/myur5.urdf.xacro (robot description, xacro)
@@ -1,11 +1,5 @@
 <?xml version="1.0"?>
 <robot xmlns:xacro="http://wiki.ros.org/xacro" name="myur5">
-    <xacro:include filename="$(find mymir_description)/urdf/mymir.urdf.xacro"/>
     <xacro:include filename="$(find booksink)/urdf/booksink.urdf"/>
-    <joint name="mir_sink_joint" type="fixed">
-        <parent link="mir/base_link"/>
-        <child link="booksink_link"/>
-        <origin xyz="-0.38478 0.285055 0.2964" rpy="0.0 0.0 0.0"/>
-    </joint>
     <link name="mass_link">
     <visual>
@@ -18,11 +12,11 @@
     </visual>
     <inertial>
-      <mass value="400"/>
+      <mass value="20"/>
       <inertia ixx="0.4" ixy="0.0" ixz="0.0" iyy="0.4" iyz="0.0" izz="0.2"/>
     </inertial>
     </link>
     <joint name="mass_joint" type="fixed">
-        <origin xyz="0 0 0.1" rpy="0.0 0.0 0.0"/>
-        <parent link="mir/base_link"/>
+        <origin xyz="0.345 -0.4 0.1" rpy="0.0 0.0 0.0"/>
+        <parent link="booksink_link"/>
         <child link="mass_link"/>
     </joint>
@@ -54,9 +48,8 @@
         <origin xyz="0 0 0" rpy="0 0 0"/>
       </joint>
-<!-- Gazebo plugin for ROS Control -->
-  <gazebo>
-    <plugin name="gazebo_ros_control" filename="libgazebo_ros_control.so">
-      <robotNamespace>/</robotNamespace>
-    </plugin>
-  </gazebo>
+    <!-- <gazebo>
+        <plugin filename="libgazebo_ros_control.so" name="gazebo_ros_control">
+            <robotNamespace>/</robotNamespace>
+        </plugin>
+    </gazebo> -->
 </robot>

File: src/myur_moveit_config/config/gazebo_myur5.urdf (robot description, URDF)
Before this commit: robot myur5, 49 links, 48 joints
Links:
- removed link mir_back_laser_link
- removed link mir_base_footprint
- removed link mir_base_link
- removed link mir_bl_caster_rotation_link
- removed link mir_bl_caster_wheel_link
- removed link mir_br_caster_rotation_link
- removed link mir_br_caster_wheel_link
- removed link mir_fl_caster_rotation_link
- removed link mir_fl_caster_wheel_link
- removed link mir_fr_caster_rotation_link
- removed link mir_fr_caster_wheel_link
- removed link mir_front_laser_link
- removed link mir_imu_frame
- removed link mir_imu_link
- removed link mir_left_wheel_link
- removed link mir_right_wheel_link
- removed link mir_surface
- removed link mir_us_1_frame
- removed link mir_us_2_frame
- link mass_link: mass 400 -> 200
Joints:
- removed joint mir_base_joint
- removed joint mir_base_link_surface_joint
- removed joint mir_base_link_to_back_laser_joint
- removed joint mir_base_link_to_front_laser_joint
- removed joint mir_base_link_to_imu_joint
- removed joint mir_bl_caster_rotation_joint
- removed joint mir_bl_caster_wheel_joint
- removed joint mir_br_caster_rotation_joint
- removed joint mir_br_caster_wheel_joint
- removed joint mir_fl_caster_rotation_joint
- removed joint mir_fl_caster_wheel_joint
- removed joint mir_fr_caster_rotation_joint
- removed joint mir_fr_caster_wheel_joint
- removed joint mir_imu_link_to_imu_frame_joint
- removed joint mir_left_wheel_joint
- removed joint mir_right_wheel_joint
- removed joint mir_sink_joint
- removed joint mir_us_1_joint
- removed joint mir_us_2_joint
- joint mass_joint: origin xyz=0 0 0.1 rpy=0.0 0.0 0.0 -> xyz=0.345 -0.4 0.1 rpy=0.0 0.0 0.0; parent mir_base_link -> booksink_link

Commit message: add separate control launch for moveit

File: src/myur_description/urdf/myur5.urdf.xacro (robot description, xacro)
@@ -12,6 +12,6 @@
     </visual>
     <inertial>
-      <mass value="20"/>
-      <inertia ixx="0.4" ixy="0.0" ixz="0.0" iyy="0.4" iyz="0.0" izz="0.2"/>
+      <mass value="200"/>
+      <inertia ixx="4.4" ixy="4.0" ixz="4.0" iyy="4.4" iyz="4.0" izz="4.2"/>
     </inertial>
     </link>

Commit message: Feb 27
Feb 27, 2024 by Cheney, Jiang Dechao

Updated package: 

	booksink
		change stl file to make it booksink closed and have larger contact are with the MiR base.

	myur_description
		This is the description package of the assembly of booksink and UR5 arm. 
		Friction coefficient has be set to be as large as the booksink won't slide on the MiR base while moving. 
		Orientation of booksink and UR5 was redesigned and now perfectly fit. 

	myur_moveit_config
		This is the package for moveit planing using myur_description, changed correspondingly with the description package. 
		NEED TO BE SOLVED: Some UR wrist can not be control by moveit.

	my_mir_control
		Contains launch files to launch both myur and MiR. Using roslaunch to launch t.launch for testing

File: src/myur_description/urdf/myur5.urdf.xacro (robot description, xacro)
@@ -7,15 +7,21 @@
         <cylinder length="0.1" radius="0.1"/>
       </geometry>
+      <surface>
+		<friction>
+		   <ode>
+		      <mu>100</mu>
+		      <mu2>100</mu2>
+	          </ode>
+		</friction>
+      </surface>
       <material name="blue">
         <color rgba="0 0 .8 1"/>
       </material>
     </visual>
-    <inertial>
-      <mass value="200"/>
-      <inertia ixx="4.4" ixy="4.0" ixz="4.0" iyy="4.4" iyz="4.0" izz="4.2"/>
-    </inertial>
+    <mass value="200" />
+    <inertial auto="true" />
     </link>
     <joint name="mass_joint" type="fixed">
-        <origin xyz="0.345 -0.4 0.1" rpy="0.0 0.0 0.0"/>
+        <origin xyz="0 0 0.1" rpy="0.0 0.0 0.0"/>
         <parent link="booksink_link"/>
         <child link="mass_link"/>
@@ -23,5 +29,5 @@
     <xacro:include filename="$(find ur_description)/urdf/ur5.xacro"/>
     <joint name="sink_ur5_joint" type="fixed">
-        <origin xyz="0.69 -0.075 0.875" rpy="0.0 0.0 0.0"/>
+        <origin xyz="-0.308 -0.2105 0.875" rpy="0.0 0.0 -1.57"/>
         <parent link="booksink_link"/>
         <child link="base_link"/>

File: src/myur_moveit_config/config/gazebo_myur5.urdf (robot description, URDF)
Before this commit: robot myur5, 30 links, 29 joints
Links:
- link mass_link: mass 200 -> None; geometry visual cylinder length=0.1 radius=0.05
Joints:
- joint mass_joint: origin xyz=0.345 -0.4 0.1 rpy=0.0 0.0 0.0 -> xyz=0 0 0.1 rpy=0.0 0.0 0.0
- joint sink_ur5_joint: origin xyz=0.69 -0.075 0.875 rpy=0.0 0.0 0.0 -> xyz=-0.308 -0.2105 0.875 rpy=0.0 0.0 -1.57
