Commit message: src
solved the shaking problems

File: src/myur_moveit_config/config/gazebo_myur5.urdf (robot description, URDF)
Before this commit: robot myur5, 24 links, 23 joints
Links:
- link left_inner_finger_pad: mass 0.1 -> None
- link right_inner_finger_pad: mass 0.1 -> None

Commit message: src
fixed the gripper shaking problem via changing the mechanical properties.

File: src/myur_moveit_config/config/gazebo_myur5.urdf (robot description, URDF)
Before this commit: robot myur5, 24 links, 23 joints
Links:
- link left_inner_finger_pad: mass None -> 0.1
- link right_inner_finger_pad: mass None -> 0.1

Commit message: modify_moveit_setting_to_adjust_the_base
solved

File: src/myur_moveit_config/config/gazebo_myur5.urdf (robot description, URDF)
Before this commit: robot myur5, 24 links, 23 joints
Links:
- removed link table
- removed link world
- added link booksink_link, mass 41.6884762061747; collision mesh filename=package://booksink/meshes/booksink_link.STL; visual mesh filename=package://booksink/meshes/booksink_link.STL
- added link camera_bottom_screw_frame
- added link camera_holder_link, mass 0.0521202445897232; collision mesh filename=package://camera_holder/meshes/camera_holder_link.STL; visual mesh filename=package://camera_holder/meshes/camera_holder_link.STL
- added link camera_link, mass 0.072; collision box size=0.02505 0.09 0.025; visual mesh filename=package://realsense2_description/meshes/d435.dae
- added link ft300_mounting_plate, mass 0.1; collision mesh filename=package://robotiq_ft_sensor/meshes/collision/mountings/robo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; visual mesh filename=package://robotiq_ft_sensor/meshes/visual/mountings/robotiq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
- added link ft300_sensor, mass 0.300; collision mesh filename=package://robotiq_ft_sensor/meshes/collision/robotiq_ft300.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; visual mesh filename=package://robotiq_ft_sensor/meshes/visual/robotiq_ft300.STL
- added link mass_link, mass 400; visual cylinder length=0.1 radius=0.1
- added link mir_back_laser_link, mass 1.2; collision mesh filename=package://mir_description/meshes/visual/sick_lms-100.stl; visual mesh filename=package://mir_description/meshes/visual/sick_lms-100.stl
- added link mir_base_footprint
- added link mir_base_link, mass 97.0; collision mesh filename=package://mir_description/meshes/collision/mir_250_base.stl; visual mesh filename=package://mir_description/meshes/visual/mir_250_base.stl
- added link mir_bl_caster_rotation_link, mass 0.3097539019; collision mesh filename=package://mir_description/meshes/collision/caster_wheel_bas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; visual mesh filename=package://mir_description/meshes/visual/caster_wheel_base.s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
- added link mir_bl_caster_wheel_link, mass 1.0; collision cylinder length=0.032 radius=0.0625; visual cylinder length=0.032 radius=0.0625
- added link mir_br_caster_rotation_link, mass 0.3097539019; collision mesh filename=package://mir_description/meshes/collision/caster_wheel_bas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; visual mesh filename=package://mir_description/meshes/visual/caster_wheel_base.s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
- added link mir_br_caster_wheel_link, mass 1.0; collision cylinder length=0.032 radius=0.0625; visual cylinder length=0.032 radius=0.0625
- added link mir_fl_caster_rotation_link, mass 0.3097539019; collision mesh filename=package://mir_description/meshes/collision/caster_wheel_bas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; visual mesh filename=package://mir_description/meshes/visual/caster_wheel_base.s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
- added link mir_fl_caster_wheel_link, mass 1.0; collision cylinder length=0.032 radius=0.0625; visual cylinder length=0.032 radius=0.0625
- added link mir_fr_caster_rotation_link, mass 0.3097539019; collision mesh filename=package://mir_description/meshes/collision/caster_wheel_bas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; visual mesh filename=package://mir_description/meshes/visual/caster_wheel_base.s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
- added link mir_fr_caster_wheel_link, mass 1.0; collision cylinder length=0.032 radius=0.0625; visual cylinder length=0.032 radius=0.0625
- added link mir_front_laser_link, mass 1.2; collision mesh filename=package://mir_description/meshes/visual/sick_lms-100.stl; visual mesh filename=package://mir_description/meshes/visual/sick_lms-100.stl
- added link mir_imu_frame
- added link mir_imu_link
- added link mir_left_wheel_link, mass 1.0; collision cylinder length=0.038 radius=0.1; visual cylinder length=0.038 radius=0.1
- added link mir_right_wheel_link, mass 1.0; collision cylinder length=0.038 radius=0.1; visual cylinder length=0.038 radius=0.1
- added link mir_surface
- added link mir_us_1_frame
- added link mir_us_2_frame
- added link robotiq_ft_frame_id
Joints:
- removed joint base_joint
- removed joint end_effector_joint
- removed joint world_joint
- added joint camera_holder_joint: type fixed, parent wrist_3_link, child camera_holder_link, origin xyz=-0.0395 0 -0.03 rpy=1.5708 0 1.5708
- added joint camera_joint: type fixed, parent camera_holder_link, child camera_bottom_screw_frame, origin xyz=-0.11 0.026 0.04 rpy=-1.5708 0 1.5708
- added joint camera_link_joint: type fixed, parent camera_bottom_screw_frame, child camera_link, origin xyz=0.010600000000000002 0.0175 0.0125 rpy=0 0 0
- added joint ft300_fix: type fixed, parent tool0, child ft300_mounting_plate, origin xyz=0 0 0 rpy=0 0 0
- added joint ft300_mounting_plate: type fixed, parent ft300_mounting_plate, child ft300_sensor, origin xyz=0 0 0.0415 rpy=0 3.141592653589793 0
- added joint ft_gripper_joint: type fixed, parent robotiq_ft_frame_id, child robotiq_arg2f_base_link, origin xyz=0 0 0 rpy=0 0 0
- added joint mass_joint: type fixed, parent mir_base_link, child mass_link, origin xyz=0 0 0.1 rpy=0.0 0.0 0.0
- added joint measurment_joint: type fixed, parent ft300_sensor, child robotiq_ft_frame_id, origin xyz=0 0 0 rpy=0 3.141592653589793 -1.5707963267948966
- added joint mir_base_joint: type fixed, parent mir_base_footprint, child mir_base_link, origin xyz=0 0 0 rpy=0 0 0
- added joint mir_base_link_surface_joint: type fixed, parent mir_base_link, child mir_surface, origin xyz=-0.004485 0 0.352 rpy=0 0 0, axis 0 0 1
- added joint mir_base_link_to_back_laser_joint: type fixed, parent mir_base_link, child mir_back_laser_link, origin xyz=-0.319485 -0.205 0.1914 rpy=0.0 0.0 -2.356194490192345
- added joint mir_base_link_to_front_laser_joint: type fixed, parent mir_base_link, child mir_front_laser_link, origin xyz=0.310515 0.205 0.1914 rpy=0.0 0.0 0.7853981633974483
- added joint mir_base_link_to_imu_joint: type fixed, parent mir_base_link, child mir_imu_link, origin xyz=0.0 0.0 0.25 rpy=0 0 0
- added joint mir_bl_caster_rotation_joint: type continuous, parent mir_base_link, child mir_bl_caster_rotation_link, origin xyz=-0.300485 0.188 0.1565 rpy=0 0 0, axis 0 0 1
- added joint mir_bl_caster_wheel_joint: type continuous, parent mir_bl_caster_rotation_link, child mir_bl_caster_wheel_link, origin xyz=-0.0382 0 -0.094 rpy=0 0 0, axis 0 1 0
- added joint mir_br_caster_rotation_joint: type continuous, parent mir_base_link, child mir_br_caster_rotation_link, origin xyz=-0.300485 -0.188 0.1565 rpy=0 0 0, axis 0 0 1
- added joint mir_br_caster_wheel_joint: type continuous, parent mir_br_caster_rotation_link, child mir_br_caster_wheel_link, origin xyz=-0.0382 0 -0.094 rpy=0 0 0, axis 0 1 0
- added joint mir_fl_caster_rotation_joint: type continuous, parent mir_base_link, child mir_fl_caster_rotation_link, origin xyz=0.299215 0.188 0.1565 rpy=0 0 0, axis 0 0 1
- added joint mir_fl_caster_wheel_joint: type continuous, parent mir_fl_caster_rotation_link, child mir_fl_caster_wheel_link, origin xyz=-0.0382 0 -0.094 rpy=0 0 0, axis 0 1 0
- added joint mir_fr_caster_rotation_joint: type continuous, parent mir_base_link, child mir_fr_caster_rotation_link, origin xyz=0.299215 -0.188 0.1565 rpy=0 0 0, axis 0 0 1
- added joint mir_fr_caster_wheel_joint: type continuous, parent mir_fr_caster_rotation_link, child mir_fr_caster_wheel_link, origin xyz=-0.0382 0 -0.094 rpy=0 0 0, axis 0 1 0
- added joint mir_imu_link_to_imu_frame_joint: type fixed, parent mir_imu_link, child mir_imu_frame, origin xyz=0 0 0 rpy=0 0 0
- added joint mir_left_wheel_joint: type continuous, parent mir_base_link, child mir_left_wheel_link, origin xyz=0.0 0.2015 0.1 rpy=0 0 0, axis 0 1 0, limit effort=100 velocity=20.0
- added joint mir_right_wheel_joint: type continuous, parent mir_base_link, child mir_right_wheel_link, origin xyz=0.0 -0.2015 0.1 rpy=0 0 0, axis 0 1 0, limit effort=100 velocity=20.0
- added joint mir_sink_joint: type fixed, parent mir_base_link, child booksink_link, origin xyz=-0.38478 0.285055 0.2964 rpy=0.0 0.0 0.0
- added joint mir_us_1_joint: type fixed, parent mir_base_link, child mir_us_1_frame, origin xyz=0.45 -0.12 0.16  rpy=0 0 0
- added joint mir_us_2_joint: type fixed, parent mir_base_link, child mir_us_2_frame, origin xyz=0.45 0.12 0.16  rpy=0 0 0
- added joint sink_ur5_joint: type fixed, parent booksink_link, child base_link, origin xyz=0.69 -0.075 0.875 rpy=0.0 0.0 0.0

Commit message: solve realsense problem
camera can work by adding some structure code in the urdf file

File: src/myur_moveit_config/config/gazebo_myur5.urdf (robot description, URDF)
Before this commit: robot myur5, 30 links, 29 joints
Links:
- added link camera_accel_frame
- added link camera_accel_optical_frame
- added link camera_color_frame
- added link camera_color_optical_frame
- added link camera_depth_frame
- added link camera_depth_optical_frame
- added link camera_gyro_frame
- added link camera_gyro_optical_frame
- added link camera_infra1_frame
- added link camera_infra1_optical_frame
- added link camera_infra2_frame
- added link camera_infra2_optical_frame
Joints:
- added joint camera_accel_joint: type fixed, parent camera_link, child camera_accel_frame, origin xyz=-0.01174 -0.00552 0.0051 rpy=0 0 0
- added joint camera_accel_optical_joint: type fixed, parent camera_accel_frame, child camera_accel_optical_frame, origin xyz=0 0 0 rpy=-1.5707963267948966 0 -1.5707963267948966
- added joint camera_color_joint: type fixed, parent camera_link, child camera_color_frame, origin xyz=0 0.015 0 rpy=0 0 0
- added joint camera_color_optical_joint: type fixed, parent camera_color_frame, child camera_color_optical_frame, origin xyz=0 0 0 rpy=-1.5707963267948966 0 -1.5707963267948966
- added joint camera_depth_joint: type fixed, parent camera_link, child camera_depth_frame, origin xyz=0 0 0 rpy=0 0 0
- added joint camera_depth_optical_joint: type fixed, parent camera_depth_frame, child camera_depth_optical_frame, origin xyz=0 0 0 rpy=-1.5707963267948966 0 -1.5707963267948966
- added joint camera_gyro_joint: type fixed, parent camera_link, child camera_gyro_frame, origin xyz=-0.01174 -0.00552 0.0051 rpy=0 0 0
- added joint camera_gyro_optical_joint: type fixed, parent camera_gyro_frame, child camera_gyro_optical_frame, origin xyz=0 0 0 rpy=-1.5707963267948966 0 -1.5707963267948966
- added joint camera_infra1_joint: type fixed, parent camera_link, child camera_infra1_frame, origin xyz=0 0.0 0 rpy=0 0 0
- added joint camera_infra1_optical_joint: type fixed, parent camera_infra1_frame, child camera_infra1_optical_frame, origin xyz=0 0 0 rpy=-1.5707963267948966 0 -1.5707963267948966
- added joint camera_infra2_joint: type fixed, parent camera_link, child camera_infra2_frame, origin xyz=0 -0.05 0 rpy=0 0 0
- added joint camera_infra2_optical_joint: type fixed, parent camera_infra2_frame, child camera_infra2_optical_frame, origin xyz=0 0 0 rpy=-1.5707963267948966 0 -1.5707963267948966
