Commit message: booksink

File: src/booksink_ur_moveit_config/config/gazebo_myur5.urdf (robot description, URDF)
Before this commit: robot myur5, 42 links, 41 joints
Links:
- link booksink_link: geometry collision mesh filename=package://booksink/meshes/booklabel.dae; visual mesh filename=package://booksink/meshes/booklabel.dae
